File: pcb/keyboard/0v1/keyboard.kicad_sch (KiCad schematic)
At the start: 0 parts

Commit message: Found footprint for the nrf52840 module.
Parts:
- added U1: 113990583, 113990583_SEE, symbol MDBT50Q-1MV2 & MDBT50Q-P1MV2:113990583
Connections:
- new net GND: U1.1 (GND), U1.15 (GND), U1.2 (GND), U1.33 (GND), U1.55 (GND)
