File: pcb/keyboard/0v1/keyboard.kicad_pcb (KiCad board)
At the start: 2 copper layers, 0 parts

Commit message: Board rules setup for PCB layouts
Other:
- rule pad_to_mask_clearance: 0 -> 0.1
Changed lines of the file:
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@@
 				(type "Bottom Silk Screen")
 			)
-			(copper_finish "None")
+			(copper_finish "HAL lead-free")
 			(dielectric_constraints no)
 		)
-		(pad_to_mask_clearance 0)
+		(pad_to_mask_clearance 0.1)
+		(solder_mask_min_width 0.1)
 		(allow_soldermask_bridges_in_footprints no)
 		(tenting front back)
