File: pcb/keyboard/v0.1/keyboard.kicad_pcb (KiCad board)
At the start: 2 copper layers, 0 parts

Commit message: Silkscreen, footprints and optional feature jumper.
Begin work on the PCB layout. For this there had to be a lot of fixes in
the footprint assignments and what gets auto populated on the Silkscreen
layer.

Also added a solder jumper for enabling optional features in the
keyboard. This will be used for bluetooth.
Parts:
- added C1: 10uf, Capacitor_SMD:C_0805_2012Metric, F.Cu at (236.0, 119.3)
- added C2: 10uf, Capacitor_SMD:C_0805_2012Metric, F.Cu at (236.0, 122.3)
- added C3: 12pF, Capacitor_SMD:C_0603_1608Metric, F.Cu at (227.7, 112.8)
- added C4: 12pF, Capacitor_SMD:C_0603_1608Metric, F.Cu at (227.7, 115.3)
- added D1: 1N4148, Diode_SMD:D_SOD-523, F.Cu at (87.5, 103.0)
- added D10: 1N4148, Diode_SMD:D_SOD-523, F.Cu at (145.1, 103.0)
- added D11: 1N4148, Diode_SMD:D_SOD-523, F.Cu at (151.5, 103.0)
- added D12: 1N4148, Diode_SMD:D_SOD-523, F.Cu at (157.9, 103.0)
- added D13: 1N4148, Diode_SMD:D_SOD-523, F.Cu at (193.3, 120.1)
- added D14: 1N4148, Diode_SMD:D_SOD-523, F.Cu at (193.3, 122.5)
- added D15: 1N4148, Diode_SMD:D_SOD-523, F.Cu at (193.3, 125.0)
- added D16: 1N4148, Diode_SMD:D_SOD-523, F.Cu at (193.3, 127.5)
- added D17: 1N4148, Diode_SMD:D_SOD-523, F.Cu at (193.3, 129.9)
- added D18: 1N4148, Diode_SMD:D_SOD-523, F.Cu at (193.3, 132.3)
- added D19: 1N4148, Diode_SMD:D_SOD-523, F.Cu at (196.9, 112.8)
- added D2: 1N4148, Diode_SMD:D_SOD-523, F.Cu at (93.9, 103.0)
- added D20: 1N4148, Diode_SMD:D_SOD-523, F.Cu at (196.9, 115.2)
- added D21: 1N4148, Diode_SMD:D_SOD-523, F.Cu at (196.9, 117.7)
- added D22: 1N4148, Diode_SMD:D_SOD-523, F.Cu at (196.9, 120.1)
- added D23: 1N4148, Diode_SMD:D_SOD-523, F.Cu at (196.9, 122.5)
- added D24: 1N4148, Diode_SMD:D_SOD-523, F.Cu at (196.9, 125.0)
- added D25: 1N4148, Diode_SMD:D_SOD-523, F.Cu at (196.9, 127.5)
- added D26: 1N4148, Diode_SMD:D_SOD-523, F.Cu at (196.9, 129.9)
- added D27: 1N4148, Diode_SMD:D_SOD-523, F.Cu at (196.9, 132.3)
- added D28: 1N4148, Diode_SMD:D_SOD-523, F.Cu at (200.5, 112.8)
- added D29: 1N4148, Diode_SMD:D_SOD-523, F.Cu at (200.5, 115.2)
- added D3: 1N4148, Diode_SMD:D_SOD-523, F.Cu at (100.3, 103.0)
- added D30: 1N4148, Diode_SMD:D_SOD-523, F.Cu at (200.5, 117.7)
- added D31: 1N4148, Diode_SMD:D_SOD-523, F.Cu at (200.5, 120.1)
- added D32: 1N4148, Diode_SMD:D_SOD-523, F.Cu at (200.5, 122.5)
- added D33: 1N4148, Diode_SMD:D_SOD-523, F.Cu at (200.5, 125.0)
- added D34: 1N4148, Diode_SMD:D_SOD-523, F.Cu at (200.5, 127.5)
- added D35: 1N4148, Diode_SMD:D_SOD-523, F.Cu at (200.5, 129.9)
- added D36: 1N4148, Diode_SMD:D_SOD-523, F.Cu at (200.5, 132.3)
- added D37: 1N4148, Diode_SMD:D_SOD-523, F.Cu at (204.1, 112.8)
- added D38: 1N4148, Diode_SMD:D_SOD-523, F.Cu at (204.1, 115.2)
- added D39: 1N4148, Diode_SMD:D_SOD-523, F.Cu at (204.1, 117.7)
- added D4: 1N4148, Diode_SMD:D_SOD-523, F.Cu at (106.7, 103.0)
- added D40: 1N4148, Diode_SMD:D_SOD-523, F.Cu at (204.1, 120.1)
- added D41: 1N4148, Diode_SMD:D_SOD-523, F.Cu at (204.1, 122.5)
- added D42: 1N4148, Diode_SMD:D_SOD-523, F.Cu at (204.1, 125.0)
- added D43: 1N4148, Diode_SMD:D_SOD-523, F.Cu at (204.1, 127.5)
- added D44: 1N4148, Diode_SMD:D_SOD-523, F.Cu at (204.1, 129.9)
- added D45: 1N4148, Diode_SMD:D_SOD-523, F.Cu at (204.1, 132.3)
- added D46: 1N4148, Diode_SMD:D_SOD-523, F.Cu at (207.7, 112.8)
- added D47: 1N4148, Diode_SMD:D_SOD-523, F.Cu at (207.7, 115.2)
- added D48: 1N4148, Diode_SMD:D_SOD-523, F.Cu at (207.7, 117.7)
- added D49: 1N4148, Diode_SMD:D_SOD-523, F.Cu at (207.7, 120.1)
- added D5: 1N4148, Diode_SMD:D_SOD-523, F.Cu at (113.1, 103.0)
- added D50: 1N4148, Diode_SMD:D_SOD-523, F.Cu at (207.7, 122.5)
- added D51: 1N4148, Diode_SMD:D_SOD-523, F.Cu at (207.7, 125.0)
- added D52: 1N4148, Diode_SMD:D_SOD-523, F.Cu at (207.7, 127.5)
- added D53: 1N4148, Diode_SMD:D_SOD-523, F.Cu at (207.7, 129.9)
- added D54: 1N4148, Diode_SMD:D_SOD-523, F.Cu at (207.7, 132.3)
- added D55: 1N4148, Diode_SMD:D_SOD-523, F.Cu at (211.3, 112.8)
- added D56: 1N4148, Diode_SMD:D_SOD-523, F.Cu at (211.3, 115.2)
- added D57: 1N4148, Diode_SMD:D_SOD-523, F.Cu at (211.3, 117.7)
- added D58: 1N4148, Diode_SMD:D_SOD-523, F.Cu at (211.3, 120.1)
- added D59: 1N4148, Diode_SMD:D_SOD-523, F.Cu at (211.3, 122.5)
- added D6: 1N4148, Diode_SMD:D_SOD-523, F.Cu at (119.5, 103.0)
- added D60: 1N4148, Diode_SMD:D_SOD-523, F.Cu at (211.3, 125.0)
- added D61: 1N4148, Diode_SMD:D_SOD-523, F.Cu at (211.3, 127.5)
- added D62: 1N4148, Diode_SMD:D_SOD-523, F.Cu at (211.3, 129.9)
- added D63: 1N4148, Diode_SMD:D_SOD-523, F.Cu at (211.3, 132.3)
- added D7: 1N4148, Diode_SMD:D_SOD-523, F.Cu at (125.9, 103.0)
- added D8: 1N4148, Diode_SMD:D_SOD-523, F.Cu at (132.3, 103.0)
- added D9: 1N4148, Diode_SMD:D_SOD-523, F.Cu at (138.7, 103.0)
- added J1: USB2.0, TH-A1OC:th_pogo_pins_4, F.Cu at (231.3, 113.1)
- added J2: SWD, TH-A1OC:th_pogo_pins_3, F.Cu at (231.3, 116.2)
- added JP1: SolderJumper_2_Open, Jumper:SolderJumper-2_P1.3mm_Open_TrianglePad1.0x1.5mm, F.Cu at (235.9, 125.6)
- added L1: 10uH, Inductor_SMD:L_0603_1608Metric, F.Cu at (227.7, 117.8)
- added R1: 2R2, Resistor_SMD:R_0603_1608Metric, F.Cu at (227.7, 120.3)
- added R2: 27R, Resistor_SMD:R_0603_1608Metric, F.Cu at (227.7, 122.8)
- added R3: 27R, Resistor_SMD:R_0603_1608Metric, F.Cu at (227.7, 125.3)
- added R4: 10K, Resistor_SMD:R_0603_1608Metric, F.Cu at (227.7, 127.8)
- added SW1: BACKTICK, TH-A1OC:tact_switch_4.5x4.5_PTS647, F.Cu at (85.0, 101.0)
- added SW10: 9, TH-A1OC:tact_switch_4.5x4.5_PTS647, F.Cu at (142.6, 101.0)
- added SW11: 0, TH-A1OC:tact_switch_4.5x4.5_PTS647, F.Cu at (149.0, 101.0)
- added SW12: BACKSPACE, TH-A1OC:tact_switch_4.5x4.5_PTS647, F.Cu at (155.4, 101.0)
- added SW13: TAB, TH-A1OC:tact_switch_4.5x4.5_PTS647, F.Cu at (197.9, 74.5)
- added SW14: Q, TH-A1OC:tact_switch_4.5x4.5_PTS647, F.Cu at (197.9, 80.9)
- added SW15: W, TH-A1OC:tact_switch_4.5x4.5_PTS647, F.Cu at (197.9, 87.3)
- added SW16: E, TH-A1OC:tact_switch_4.5x4.5_PTS647, F.Cu at (197.9, 93.8)
- added SW17: R, TH-A1OC:tact_switch_4.5x4.5_PTS647, F.Cu at (197.9, 100.2)
- added SW18: T, TH-A1OC:tact_switch_4.5x4.5_PTS647, F.Cu at (197.9, 106.7)
- added SW19: Y, TH-A1OC:tact_switch_4.5x4.5_PTS647, F.Cu at (206.3, 55.1)
- added SW2: 1, TH-A1OC:tact_switch_4.5x4.5_PTS647, F.Cu at (91.4, 101.0)
- added SW20: U, TH-A1OC:tact_switch_4.5x4.5_PTS647, F.Cu at (206.3, 61.5)
- added SW21: I, TH-A1OC:tact_switch_4.5x4.5_PTS647, F.Cu at (206.3, 68.0)
- added SW22: O, TH-A1OC:tact_switch_4.5x4.5_PTS647, F.Cu at (206.3, 74.5)
- added SW23: P, TH-A1OC:tact_switch_4.5x4.5_PTS647, F.Cu at (206.3, 80.9)
- added SW24: RETURN, TH-A1OC:tact_switch_4.5x4.5_PTS647, F.Cu at (206.3, 87.3)
- added SW25: CAPS, TH-A1OC:tact_switch_4.5x4.5_PTS647, F.Cu at (206.3, 93.8)
- added SW26: A, TH-A1OC:tact_switch_4.5x4.5_PTS647, F.Cu at (206.3, 100.2)
- added SW27: S, TH-A1OC:tact_switch_4.5x4.5_PTS647, F.Cu at (206.3, 106.7)
- added SW28: D, TH-A1OC:tact_switch_4.5x4.5_PTS647, F.Cu at (214.7, 55.1)
- added SW29: F, TH-A1OC:tact_switch_4.5x4.5_PTS647, F.Cu at (214.7, 61.5)
- added SW3: 2, TH-A1OC:tact_switch_4.5x4.5_PTS647, F.Cu at (97.8, 101.0)
- added SW30: G, TH-A1OC:tact_switch_4.5x4.5_PTS647, F.Cu at (214.7, 68.0)
- added SW31: H, TH-A1OC:tact_switch_4.5x4.5_PTS647, F.Cu at (214.7, 74.5)
- added SW32: J, TH-A1OC:tact_switch_4.5x4.5_PTS647, F.Cu at (214.7, 80.9)
- added SW33: K, TH-A1OC:tact_switch_4.5x4.5_PTS647, F.Cu at (214.7, 87.3)
- added SW34: L, TH-A1OC:tact_switch_4.5x4.5_PTS647, F.Cu at (214.7, 93.8)
- added SW35: SEMI, TH-A1OC:tact_switch_4.5x4.5_PTS647, F.Cu at (214.7, 100.2)
- added SW36: QUOTE, TH-A1OC:tact_switch_4.5x4.5_PTS647, F.Cu at (214.7, 106.7)
- added SW37: LSHIFT, TH-A1OC:tact_switch_4.5x4.5_PTS647, F.Cu at (223.1, 55.1)
- added SW38: Z, TH-A1OC:tact_switch_4.5x4.5_PTS647, F.Cu at (223.1, 61.5)
- added SW39: X, TH-A1OC:tact_switch_4.5x4.5_PTS647, F.Cu at (223.1, 68.0)
- added SW4: 3, TH-A1OC:tact_switch_4.5x4.5_PTS647, F.Cu at (104.2, 101.0)
- added SW40: C, TH-A1OC:tact_switch_4.5x4.5_PTS647, F.Cu at (223.1, 74.5)
- added SW41: V, TH-A1OC:tact_switch_4.5x4.5_PTS647, F.Cu at (223.1, 80.9)
- added SW42: B, TH-A1OC:tact_switch_4.5x4.5_PTS647, F.Cu at (223.1, 87.3)
- added SW43: N, TH-A1OC:tact_switch_4.5x4.5_PTS647, F.Cu at (223.1, 93.8)
- added SW44: M, TH-A1OC:tact_switch_4.5x4.5_PTS647, F.Cu at (223.1, 100.2)
- added SW45: COMMA, TH-A1OC:tact_switch_4.5x4.5_PTS647, F.Cu at (223.1, 106.7)
- added SW46: DOT, TH-A1OC:tact_switch_4.5x4.5_PTS647, F.Cu at (231.5, 55.1)
- added SW47: QUEST, TH-A1OC:tact_switch_4.5x4.5_PTS647, F.Cu at (231.5, 61.5)
- added SW48: RSHIFT, TH-A1OC:tact_switch_4.5x4.5_PTS647, F.Cu at (231.5, 68.0)
- added SW49: FN, TH-A1OC:tact_switch_4.5x4.5_PTS647, F.Cu at (231.5, 74.5)
- added SW5: 4, TH-A1OC:tact_switch_4.5x4.5_PTS647, F.Cu at (110.6, 101.0)
- added SW50: LCTRL, TH-A1OC:tact_switch_4.5x4.5_PTS647, F.Cu at (231.5, 80.9)
- added SW51: LSUPER, TH-A1OC:tact_switch_4.5x4.5_PTS647, F.Cu at (231.5, 87.3)
- added SW52: LALT, TH-A1OC:tact_switch_4.5x4.5_PTS647, F.Cu at (231.5, 93.8)
- added SW53: SPACE, TH-A1OC:tact_switch_4.5x4.5_PTS647, F.Cu at (231.5, 100.2)
- added SW54: RALT, TH-A1OC:tact_switch_4.5x4.5_PTS647, F.Cu at (231.5, 106.7)
- added SW55: RSUPER, TH-A1OC:tact_switch_4.5x4.5_PTS647, F.Cu at (239.9, 55.1)
- added SW56: MENU, TH-A1OC:tact_switch_4.5x4.5_PTS647, F.Cu at (239.9, 61.5)
- added SW57: RCTRL, TH-A1OC:tact_switch_4.5x4.5_PTS647, F.Cu at (239.9, 68.0)
- added SW58: C1, TH-A1OC:tact_switch_4.5x4.5_PTS647, F.Cu at (239.9, 74.5)
- added SW59: C2, TH-A1OC:tact_switch_4.5x4.5_PTS647, F.Cu at (239.9, 80.9)
- added SW6: 5, TH-A1OC:tact_switch_4.5x4.5_PTS647, F.Cu at (117.0, 101.0)
- added SW60: C3, TH-A1OC:tact_switch_4.5x4.5_PTS647, F.Cu at (239.9, 87.3)
- added SW61: C4, TH-A1OC:tact_switch_4.5x4.5_PTS647, F.Cu at (239.9, 93.8)
- added SW62: C5, TH-A1OC:tact_switch_4.5x4.5_PTS647, F.Cu at (239.9, 100.2)
- added SW63: C6, TH-A1OC:tact_switch_4.5x4.5_PTS647, F.Cu at (239.9, 106.7)
- added SW7: 6, TH-A1OC:tact_switch_4.5x4.5_PTS647, F.Cu at (123.4, 101.0)
- added SW8: 7, TH-A1OC:tact_switch_4.5x4.5_PTS647, F.Cu at (129.8, 101.0)
- added SW9: 8, TH-A1OC:tact_switch_4.5x4.5_PTS647, F.Cu at (136.2, 101.0)
- added TP1: TestPoint, TestPoint:TestPoint_Pad_D2.0mm, F.Cu at (231.8, 119.8)
- added TP2: TestPoint, TestPoint:TestPoint_Pad_D2.0mm, F.Cu at (231.8, 123.9)
- added U1: MDBT50Q-P1MV2, TH-A1OC:TH_MDBT50Q-P1MV2, F.Cu at (213.8, 112.3)
- added Y1: 32.768, Crystal:Crystal_SMD_3215-2Pin_3.2x1.5mm, F.Cu at (240.8, 119.5)
Routing:
- net /SOURCE1: track 0.00 -> 161.2 mm
- net Net-(D4-A): track 0.00 -> 7.30 mm
- net Net-(D3-A): track 0.00 -> 7.30 mm
- net Net-(D5-A): track 0.00 -> 7.29 mm
- net Net-(D6-A): track 0.00 -> 7.27 mm
- net Net-(D1-A): track 0.00 -> 7.27 mm
- net Net-(D12-A): track 0.00 -> 7.26 mm
- net Net-(D11-A): track 0.00 -> 7.26 mm
- net Net-(D9-A): track 0.00 -> 7.26 mm
- net Net-(D8-A): track 0.00 -> 7.26 mm
- net Net-(D7-A): track 0.00 -> 7.25 mm
- net Net-(D10-A): track 0.00 -> 7.25 mm
- net Net-(D2-A): track 0.00 -> 2.05 mm
Other:
- board outline added: 80 x 50 mm
