File: pcb/keyboard/v0.1/keyboard.kicad_sch (KiCad schematic)
At the start: 140 parts, among them SW1 A, SW10 A, SW11 A, SW12 A, SW13 A, SW14 A, SW15 A, SW16 A, SW17 A, SW18 A, SW19 A, SW2 A, SW20 A, SW21 A, SW22 A, SW23 A, SW24 A, SW25 A, SW26 A, SW27 A, SW28 A, SW29 A, SW3 A, SW30 A, SW31 A, SW32 A, SW33 A, SW34 A, SW35 A, SW36 A, SW37 A, SW38 A, SW39 A, SW4 A, SW40 A, SW41 A, SW42 A, SW43 A, SW44 A, SW45 A, SW46 A, SW47 A, SW48 A, SW49 A, SW5 A, SW50 A, SW51 A, SW52 A, SW53 A, SW54 A, SW55 A, SW56 A, SW57 A, SW58 A, SW59 A, SW6 A, SW60 A, SW61 A, SW62 A, SW63 A, SW7 A, SW8 A, SW9 A, U1 MDBT50Q-P1MV2, Y1 32.768

Commit message: Forgot to assign footprints for previous commit
Parts:
- J1: footprint (none) -> TH-A1OC:th_pogo_pins_4
- J2: renamed from J3; footprint (none) -> TH-A1OC:th_pogo_pins_3
- SW1, SW10, SW11, SW12, SW13, SW14, SW15, SW16, SW17, SW18, SW19, SW2, SW20, SW21, SW22, SW23, SW24, SW25, SW26, SW27, SW28, SW29, SW3, SW30, SW31, SW32, SW33, SW34, SW35, SW36, SW37, SW38, SW39, SW4, SW40, SW41, SW42, SW43, SW44, SW45, SW46, SW47, SW48, SW49, SW50, SW51, SW52, SW53, SW54, SW55, SW56, SW57, SW58, SW59, SW6, SW60, SW61, SW62, SW63, SW7, SW8, SW9: footprint (none) -> TH-A1OC:tact_switch_4.5x4.5_PTS647
Changed lines of the file:
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@@
 			)
 		)
-		(property "Footprint" ""
+		(property "Footprint" "TH-A1OC:tact_switch_4.5x4.5_PTS647"
 			(at 256.54 231.14 0)
 			(effects
@@
 			)
 		)
-		(property "Footprint" ""
+		(property "Footprint" "TH-A1OC:tact_switch_4.5x4.5_PTS647"
 			(at 218.44 332.74 0)
 			(effects
@@
 			)
 		)
-		(property "Footprint" ""
+		(property "Footprint" "TH-A1OC:tact_switch_4.5x4.5_PTS647"
 			(at 180.34 281.94 0)
 			(effects
@@
 			)
 		)
-		(property "Footprint" ""
+		(property "Footprint" "TH-A1OC:tact_switch_4.5x4.5_PTS647"
 			(at 370.84 332.74 0)
 			(effects
@@
 			)
 		)
-		(property "Footprint" ""
+		(property "Footprint" "TH-A1OC:tact_switch_4.5x4.5_PTS647"
 			(at 281.94 256.54 0)
 			(effects
@@
 			)
 		)
-		(property "Footprint" ""
+		(property "Footprint" "TH-A1OC:tact_switch_4.5x4.5_PTS647"
 			(at 358.14 281.94 0)
 			(effects
@@
 			)
 		)
-		(property "Footprint" ""
+		(property "Footprint" "TH-A1OC:tact_switch_4.5x4.5_PTS647"
 			(at 408.94 231.14 0)
 			(effects
@@
 			)
 		)
-		(property "Footprint" ""
+		(property "Footprint" "TH-A1OC:tact_switch_4.5x4.5_PTS647"
 			(at 205.74 256.54 0)
 			(effects
@@
 			)
 		)
-		(property "Footprint" ""
+		(property "Footprint" "TH-A1OC:tact_switch_4.5x4.5_PTS647"
 			(at 256.54 256.54 0)
 			(effects
@@
 			)
 		)
-		(property "Footprint" ""
+		(property "Footprint" "TH-A1OC:tact_switch_4.5x4.5_PTS647"
 			(at 383.54 307.34 0)
 			(effects
@@
 			)
 		)
-		(property "Footprint" ""
+		(property "Footprint" "TH-A1OC:tact_switch_4.5x4.5_PTS647"
 			(at 408.94 281.94 0)
 			(effects
@@
 			)
 		)
-		(property "Footprint" ""
+		(property "Footprint" "TH-A1OC:tact_switch_4.5x4.5_PTS647"
 			(at 154.94 256.54 0)
 			(effects
@@
 			)
 		)
-		(property "Footprint" ""
+		(property "Footprint" "TH-A1OC:tact_switch_4.5x4.5_PTS647"
 			(at 408.94 205.74 0)
 			(effects
@@
 			)
 		)
-		(property "Footprint" ""
+		(property "Footprint" "TH-A1OC:tact_switch_4.5x4.5_PTS647"
 			(at 383.54 205.74 0)
 			(effects
@@
 			)
 		)
-		(property "Footprint" ""
+		(property "Footprint" "TH-A1OC:tact_switch_4.5x4.5_PTS647"
 			(at 321.31 332.74 0)
 			(effects
@@
 			)
 		)
-		(property "Footprint" ""
+		(property "Footprint" "TH-A1OC:tact_switch_4.5x4.5_PTS647"
 			(at 294.64 307.34 0)
 			(effects
@@
 			)
 		)
-		(property "Footprint" ""
+		(property "Footprint" "TH-A1OC:tact_switch_4.5x4.5_PTS647"
 			(at 231.14 256.54 0)
 			(effects
@@
 			)
 		)
-		(property "Footprint" ""
+		(property "Footprint" "TH-A1OC:th_pogo_pins_4"
 			(at 471.17 27.94 0)
 			(effects
@@
 			)
 		)
-		(property "Footprint" ""
+		(property "Footprint" "TH-A1OC:tact_switch_4.5x4.5_PTS647"
 			(at 358.14 205.74 0)
 			(effects
@@
 			)
 		)
-		(property "Footprint" ""
+		(property "Footprint" "TH-A1OC:tact_switch_4.5x4.5_PTS647"
 			(at 307.34 231.14 0)
 			(effects
@@
 			)
 		)
-		(property "Footprint" ""
+		(property "Footprint" "TH-A1OC:tact_switch_4.5x4.5_PTS647"
 			(at 205.74 205.74 0)
 			(effects
@@
 			)
 		)
-		(property "Footprint" ""
+		(property "Footprint" "TH-A1OC:tact_switch_4.5x4.5_PTS647"
 			(at 332.74 281.94 0)
 			(effects
@@
 			)
 		)
-		(property "Footprint" ""
+		(property "Footprint" "TH-A1OC:tact_switch_4.5x4.5_PTS647"
 			(at 332.74 231.14 0)
 			(effects
@@
 			)
 		)
-		(property "Footprint" ""
+		(property "Footprint" "TH-A1OC:tact_switch_4.5x4.5_PTS647"
 			(at 205.74 307.34 0)
 			(effects
@@
 			)
 		)
-		(property "Footprint" ""
+		(property "Footprint" "TH-A1OC:tact_switch_4.5x4.5_PTS647"
 			(at 154.94 307.34 0)
 			(effects
@@
 			)
 		)
-		(property "Footprint" ""
+		(property "Footprint" "TH-A1OC:tact_switch_4.5x4.5_PTS647"
 			(at 383.54 281.94 0)
 			(effects
@@
 			)
 		)
-		(property "Footprint" ""
+		(property "Footprint" "TH-A1OC:tact_switch_4.5x4.5_PTS647"
 			(at 231.14 281.94 0)
 			(effects
@@
 			)
 		)
-		(property "Footprint" ""
+		(property "Footprint" "TH-A1OC:tact_switch_4.5x4.5_PTS647"
 			(at 180.34 205.74 0)
 			(effects
@@
 			)
 		)
-		(property "Footprint" ""
+		(property "Footprint" "TH-A1OC:tact_switch_4.5x4.5_PTS647"
 			(at 180.34 231.14 0)
 			(effects
@@
 			)
 		)
-		(property "Footprint" ""
+		(property "Footprint" "TH-A1OC:tact_switch_4.5x4.5_PTS647"
 			(at 180.34 307.34 0)
 			(effects
@@
 			)
 		)
-		(property "Footprint" ""
+		(property "Footprint" "TH-A1OC:tact_switch_4.5x4.5_PTS647"
 			(at 408.94 256.54 0)
 			(effects
@@
 			)
 		)
-		(property "Footprint" ""
+		(property "Footprint" "TH-A1OC:tact_switch_4.5x4.5_PTS647"
 			(at 358.14 256.54 0)
 			(effects
@@
 			)
 		)
-		(property "Footprint" ""
+		(property "Footprint" "TH-A1OC:tact_switch_4.5x4.5_PTS647"
 			(at 231.14 307.34 0)
 			(effects
@@
 			)
 		)
-		(property "Footprint" ""
+		(property "Footprint" "TH-A1OC:tact_switch_4.5x4.5_PTS647"
 			(at 256.54 281.94 0)
 			(effects
@@
 			)
 		)
-		(property "Footprint" ""
+		(property "Footprint" "TH-A1OC:tact_switch_4.5x4.5_PTS647"
 			(at 205.74 231.14 0)
 			(effects
@@
 			)
 		)
-		(property "Footprint" ""
+		(property "Footprint" "TH-A1OC:tact_switch_4.5x4.5_PTS647"
 			(at 421.64 332.74 0)
 			(effects
@@
 			)
 		)
-		(property "Footprint" ""
+		(property "Footprint" "TH-A1OC:tact_switch_4.5x4.5_PTS647"
 			(at 358.14 307.34 0)
 			(effects
@@
 			)
 		)
-		(property "Footprint" ""
+		(property "Footprint" "TH-A1OC:tact_switch_4.5x4.5_PTS647"
 			(at 281.94 281.94 0)
 			(effects
@@
 			)
 		)
-		(property "Footprint" ""
+		(property "Footprint" "TH-A1OC:tact_switch_4.5x4.5_PTS647"
 			(at 358.14 231.14 0)
 			(effects
@@
 			)
 		)
-		(property "Footprint" ""
+		(property "Footprint" "TH-A1OC:tact_switch_4.5x4.5_PTS647"
 			(at 434.34 231.14 0)
 			(effects
@@
 			)
 		)
-		(property "Footprint" ""
+		(property "Footprint" "TH-A1OC:tact_switch_4.5x4.5_PTS647"
 			(at 307.34 281.94 0)
 			(effects
@@
 			)
 		)
-		(property "Footprint" ""
+		(property "Footprint" "TH-A1OC:tact_switch_4.5x4.5_PTS647"
 			(at 383.54 256.54 0)
 			(effects
@@
 			)
 		)
-		(property "Footprint" ""
+		(property "Footprint" "TH-A1OC:tact_switch_4.5x4.5_PTS647"
 			(at 269.24 332.74 0)
 			(effects
@@
 			)
 		)
-		(property "Footprint" ""
+		(property "Footprint" "TH-A1OC:tact_switch_4.5x4.5_PTS647"
 			(at 307.34 205.74 0)
 			(effects
@@
 			)
 		)
-		(property "Footprint" ""
+		(property "Footprint" "TH-A1OC:tact_switch_4.5x4.5_PTS647"
 			(at 307.34 256.54 0)
 			(effects
@@
 			)
 		)
-		(property "Footprint" ""
+		(property "Footprint" "TH-A1OC:tact_switch_4.5x4.5_PTS647"
 			(at 180.34 256.54 0)
 			(effects
@@
 			)
 		)
-		(property "Footprint" ""
+		(property "Footprint" "TH-A1OC:tact_switch_4.5x4.5_PTS647"
 			(at 167.64 332.74 0)
 			(effects
@@
 			)
 		)
-		(property "Footprint" ""
+		(property "Footprint" "TH-A1OC:tact_switch_4.5x4.5_PTS647"
 			(at 434.34 205.74 0)
 			(effects
@@
 			)
 		)
-		(property "Footprint" ""
+		(property "Footprint" "TH-A1OC:tact_switch_4.5x4.5_PTS647"
 			(at 154.94 231.14 0)
 			(effects
@@
 			)
 		)
-		(property "Footprint" ""
+		(property "Footprint" "TH-A1OC:tact_switch_4.5x4.5_PTS647"
 			(at 231.14 205.74 0)
 			(effects
@@
 			)
 		)
-		(property "Footprint" ""
+		(property "Footprint" "TH-A1OC:tact_switch_4.5x4.5_PTS647"
 			(at 434.34 281.94 0)
 			(effects
@@
 			)
 		)
-		(property "Footprint" ""
+		(property "Footprint" "TH-A1OC:tact_switch_4.5x4.5_PTS647"
 			(at 205.74 281.94 0)
 			(effects
@@
 			)
 		)
-		(property "Footprint" ""
+		(property "Footprint" "TH-A1OC:tact_switch_4.5x4.5_PTS647"
 			(at 434.34 307.34 0)
 			(effects
@@
 			)
 		)
-		(property "Footprint" ""
+		(property "Footprint" "TH-A1OC:tact_switch_4.5x4.5_PTS647"
 			(at 256.54 205.74 0)
 			(effects
@@
 			)
 		)
-		(property "Footprint" ""
+		(property "Footprint" "TH-A1OC:tact_switch_4.5x4.5_PTS647"
 			(at 281.94 205.74 0)
 			(effects
@@
 			)
 		)
-		(property "Footprint" ""
+		(property "Footprint" "TH-A1OC:tact_switch_4.5x4.5_PTS647"
 			(at 281.94 231.14 0)
 			(effects
@@
 			)
 		)
-		(property "Footprint" ""
+		(property "Footprint" "TH-A1OC:tact_switch_4.5x4.5_PTS647"
 			(at 332.74 256.54 0)
 			(effects
@@
 			)
 		)
-		(property "Footprint" ""
+		(property "Footprint" "TH-A1OC:tact_switch_4.5x4.5_PTS647"
 			(at 434.34 256.54 0)
 			(effects
@@
 			)
 		)
-		(property "Footprint" ""
+		(property "Footprint" "TH-A1OC:tact_switch_4.5x4.5_PTS647"
 			(at 231.14 231.14 0)
 			(effects
@@
 		(dnp no)
 		(fields_autoplaced yes)
-		(property "Reference" "J3"
+		(property "Reference" "J2"
 			(at 505.46 31.7499 0)
 			(effects
@@
 			)
 		)
-		(property "Footprint" ""
+		(property "Footprint" "TH-A1OC:th_pogo_pins_3"
 			(at 491.49 27.94 0)
 			(effects
@@
 			(project ""
 				(path "/c19feaf6-aecc-4469-9f12-5cd065a0782d"
-					(reference "J3")
+					(reference "J2")
 					(unit 1)
 				)
@@
 			)
 		)
-		(property "Footprint" ""
+		(property "Footprint" "TH-A1OC:tact_switch_4.5x4.5_PTS647"
 			(at 154.94 281.94 0)
 			(effects
@@
 			)
 		)
-		(property "Footprint" ""
+		(property "Footprint" "TH-A1OC:tact_switch_4.5x4.5_PTS647"
 			(at 332.74 205.74 0)
 			(effects
@@
 			)
 		)
-		(property "Footprint" ""
+		(property "Footprint" "TH-A1OC:tact_switch_4.5x4.5_PTS647"
 			(at 383.54 231.14 0)
 			(effects
@@
 			)
 		)
-		(property "Footprint" ""
+		(property "Footprint" "TH-A1OC:tact_switch_4.5x4.5_PTS647"
 			(at 408.94 307.34 0)
 			(effects

Commit message: Silkscreen, footprints and optional feature jumper.
Begin work on the PCB layout. For this there had to be a lot of fixes in
the footprint assignments and what gets auto populated on the Silkscreen
layer.

Also added a solder jumper for enabling optional features in the
keyboard. This will be used for bluetooth.
Parts:
- removed SW1, SW10, SW11, SW12, SW13, SW14, SW15, SW16, SW17, SW18, SW19, SW2, SW20, SW21, SW22, SW23, SW24, SW25, SW26, SW27, SW28, SW29, SW3, SW30, SW31, SW32, SW33, SW34, SW35, SW36, SW37, SW38, SW39, SW4, SW40, SW41, SW42, SW43, SW44, SW45, SW46, SW47, SW48, SW49, SW5, SW50, SW51, SW52, SW53, SW54, SW55, SW56, SW57, SW58, SW59, SW6, SW60, SW61, SW62, SW63, SW7, SW8, SW9: A, TH-A1OC:tact_switch_4.5x4.5_PTS647, symbol Switch:SW_Push_45deg
- added JP1: SolderJumper_2_Open, Jumper:SolderJumper-2_P1.3mm_Open_TrianglePad1.0x1.5mm, symbol Jumper:SolderJumper_2_Open
- added R4: 10K, Resistor_SMD:R_0603_1608Metric, symbol Device:R
- added SW1: BACKTICK, TH-A1OC:tact_switch_4.5x4.5_PTS647, symbol TH-A10C:SW_Push_45deg
- added SW10: 9, TH-A1OC:tact_switch_4.5x4.5_PTS647, symbol TH-A10C:SW_Push_45deg
- added SW11: 0, TH-A1OC:tact_switch_4.5x4.5_PTS647, symbol TH-A10C:SW_Push_45deg
- added SW12: BACKSPACE, TH-A1OC:tact_switch_4.5x4.5_PTS647, symbol TH-A10C:SW_Push_45deg
- added SW13: TAB, TH-A1OC:tact_switch_4.5x4.5_PTS647, symbol TH-A10C:SW_Push_45deg
- added SW14: Q, TH-A1OC:tact_switch_4.5x4.5_PTS647, symbol TH-A10C:SW_Push_45deg
- added SW15: W, TH-A1OC:tact_switch_4.5x4.5_PTS647, symbol TH-A10C:SW_Push_45deg
- added SW16: E, TH-A1OC:tact_switch_4.5x4.5_PTS647, symbol TH-A10C:SW_Push_45deg
- added SW17: R, TH-A1OC:tact_switch_4.5x4.5_PTS647, symbol TH-A10C:SW_Push_45deg
- added SW18: T, TH-A1OC:tact_switch_4.5x4.5_PTS647, symbol TH-A10C:SW_Push_45deg
- added SW19: Y, TH-A1OC:tact_switch_4.5x4.5_PTS647, symbol TH-A10C:SW_Push_45deg
- added SW2: 1, TH-A1OC:tact_switch_4.5x4.5_PTS647, symbol TH-A10C:SW_Push_45deg
- added SW20: U, TH-A1OC:tact_switch_4.5x4.5_PTS647, symbol TH-A10C:SW_Push_45deg
- added SW21: I, TH-A1OC:tact_switch_4.5x4.5_PTS647, symbol TH-A10C:SW_Push_45deg
- added SW22: O, TH-A1OC:tact_switch_4.5x4.5_PTS647, symbol TH-A10C:SW_Push_45deg
- added SW23: P, TH-A1OC:tact_switch_4.5x4.5_PTS647, symbol TH-A10C:SW_Push_45deg
- added SW24: RETURN, TH-A1OC:tact_switch_4.5x4.5_PTS647, symbol TH-A10C:SW_Push_45deg
- added SW25: CAPS, TH-A1OC:tact_switch_4.5x4.5_PTS647, symbol TH-A10C:SW_Push_45deg
- added SW26: A, TH-A1OC:tact_switch_4.5x4.5_PTS647, symbol TH-A10C:SW_Push_45deg
- added SW27: S, TH-A1OC:tact_switch_4.5x4.5_PTS647, symbol TH-A10C:SW_Push_45deg
- added SW28: D, TH-A1OC:tact_switch_4.5x4.5_PTS647, symbol TH-A10C:SW_Push_45deg
- added SW29: F, TH-A1OC:tact_switch_4.5x4.5_PTS647, symbol TH-A10C:SW_Push_45deg
- added SW3: 2, TH-A1OC:tact_switch_4.5x4.5_PTS647, symbol TH-A10C:SW_Push_45deg
- added SW30: G, TH-A1OC:tact_switch_4.5x4.5_PTS647, symbol TH-A10C:SW_Push_45deg
- added SW31: H, TH-A1OC:tact_switch_4.5x4.5_PTS647, symbol TH-A10C:SW_Push_45deg
- added SW32: J, TH-A1OC:tact_switch_4.5x4.5_PTS647, symbol TH-A10C:SW_Push_45deg
- added SW33: K, TH-A1OC:tact_switch_4.5x4.5_PTS647, symbol TH-A10C:SW_Push_45deg
- added SW34: L, TH-A1OC:tact_switch_4.5x4.5_PTS647, symbol TH-A10C:SW_Push_45deg
- added SW35: SEMI, TH-A1OC:tact_switch_4.5x4.5_PTS647, symbol TH-A10C:SW_Push_45deg
- added SW36: QUOTE, TH-A1OC:tact_switch_4.5x4.5_PTS647, symbol TH-A10C:SW_Push_45deg
- added SW37: LSHIFT, TH-A1OC:tact_switch_4.5x4.5_PTS647, symbol TH-A10C:SW_Push_45deg
- added SW38: Z, TH-A1OC:tact_switch_4.5x4.5_PTS647, symbol TH-A10C:SW_Push_45deg
- added SW39: X, TH-A1OC:tact_switch_4.5x4.5_PTS647, symbol TH-A10C:SW_Push_45deg
- added SW4: 3, TH-A1OC:tact_switch_4.5x4.5_PTS647, symbol TH-A10C:SW_Push_45deg
- added SW40: C, TH-A1OC:tact_switch_4.5x4.5_PTS647, symbol TH-A10C:SW_Push_45deg
- added SW41: V, TH-A1OC:tact_switch_4.5x4.5_PTS647, symbol TH-A10C:SW_Push_45deg
- added SW42: B, TH-A1OC:tact_switch_4.5x4.5_PTS647, symbol TH-A10C:SW_Push_45deg
- added SW43: N, TH-A1OC:tact_switch_4.5x4.5_PTS647, symbol TH-A10C:SW_Push_45deg
- added SW44: M, TH-A1OC:tact_switch_4.5x4.5_PTS647, symbol TH-A10C:SW_Push_45deg
- added SW45: COMMA, TH-A1OC:tact_switch_4.5x4.5_PTS647, symbol TH-A10C:SW_Push_45deg
- added SW46: DOT, TH-A1OC:tact_switch_4.5x4.5_PTS647, symbol TH-A10C:SW_Push_45deg
- added SW47: QUEST, TH-A1OC:tact_switch_4.5x4.5_PTS647, symbol TH-A10C:SW_Push_45deg
- added SW48: RSHIFT, TH-A1OC:tact_switch_4.5x4.5_PTS647, symbol TH-A10C:SW_Push_45deg
- added SW49: FN, TH-A1OC:tact_switch_4.5x4.5_PTS647, symbol TH-A10C:SW_Push_45deg
- added SW5: 4, TH-A1OC:tact_switch_4.5x4.5_PTS647, symbol TH-A10C:SW_Push_45deg
- added SW50: LCTRL, TH-A1OC:tact_switch_4.5x4.5_PTS647, symbol TH-A10C:SW_Push_45deg
- added SW51: LSUPER, TH-A1OC:tact_switch_4.5x4.5_PTS647, symbol TH-A10C:SW_Push_45deg
- added SW52: LALT, TH-A1OC:tact_switch_4.5x4.5_PTS647, symbol TH-A10C:SW_Push_45deg
- added SW53: SPACE, TH-A1OC:tact_switch_4.5x4.5_PTS647, symbol TH-A10C:SW_Push_45deg
- added SW54: RALT, TH-A1OC:tact_switch_4.5x4.5_PTS647, symbol TH-A10C:SW_Push_45deg
- added SW55: RSUPER, TH-A1OC:tact_switch_4.5x4.5_PTS647, symbol TH-A10C:SW_Push_45deg
- added SW56: MENU, TH-A1OC:tact_switch_4.5x4.5_PTS647, symbol TH-A10C:SW_Push_45deg
- added SW57: RCTRL, TH-A1OC:tact_switch_4.5x4.5_PTS647, symbol TH-A10C:SW_Push_45deg
- added SW58: C1, TH-A1OC:tact_switch_4.5x4.5_PTS647, symbol TH-A10C:SW_Push_45deg
- added SW59: C2, TH-A1OC:tact_switch_4.5x4.5_PTS647, symbol TH-A10C:SW_Push_45deg
- added SW6: 5, TH-A1OC:tact_switch_4.5x4.5_PTS647, symbol TH-A10C:SW_Push_45deg
- added SW60: C3, TH-A1OC:tact_switch_4.5x4.5_PTS647, symbol TH-A10C:SW_Push_45deg
- added SW61: C4, TH-A1OC:tact_switch_4.5x4.5_PTS647, symbol TH-A10C:SW_Push_45deg
- added SW62: C5, TH-A1OC:tact_switch_4.5x4.5_PTS647, symbol TH-A10C:SW_Push_45deg
- added SW63: C6, TH-A1OC:tact_switch_4.5x4.5_PTS647, symbol TH-A10C:SW_Push_45deg
- added SW7: 6, TH-A1OC:tact_switch_4.5x4.5_PTS647, symbol TH-A10C:SW_Push_45deg
- added SW8: 7, TH-A1OC:tact_switch_4.5x4.5_PTS647, symbol TH-A10C:SW_Push_45deg
- added SW9: 8, TH-A1OC:tact_switch_4.5x4.5_PTS647, symbol TH-A10C:SW_Push_45deg
- J1: value ~ -> USB2.0
- J2: value ~ -> SWD
- U1: footprint (none) -> TH-A1OC:TH_MDBT50Q-P1MV2
- renumbered D5 to D1, D1 to D2, D2 to D3, D3 to D4, D4 to D5
Connections:
- net GND: now also JP1.1 (A)
- net SOURCE1: now also SW1.1, SW10.1, SW11.1, SW12.1, SW2.1, SW3.1, SW4.1, SW5.1, SW6.1, SW7.1, SW8.1, SW9.1
- net SOURCE2: now also SW13.1, SW14.1, SW15.1, SW16.1, SW17.1, SW18.1, SW19.1, SW20.1, SW21.1, SW22.1, SW23.1, SW24.1
- net SOURCE3: now also SW25.1, SW26.1, SW27.1, SW28.1, SW29.1, SW30.1, SW31.1, SW32.1, SW33.1, SW34.1, SW35.1, SW36.1
- net SOURCE4: now also SW37.1, SW38.1, SW39.1, SW40.1, SW41.1, SW42.1, SW43.1, SW44.1, SW45.1, SW46.1, SW47.1, SW48.1
- net SOURCE5: now also SW49.1, SW50.1, SW51.1, SW52.1, SW53.1, SW54.1, SW55.1, SW56.1, SW57.1
- net SOURCE6: now also SW58.1, SW59.1, SW60.1, SW61.1, SW62.1, SW63.1
- net at D17.2 (A): now also SW17.2
- net at D59.2 (A): now also SW59.2
- net at D51.2 (A): now also SW51.2
- net at D9.2 (A): now also SW9.2
- net at D2.2 (A): now also SW2.2
- net at D38.2 (A): now also SW38.2
- net at D62.2 (A): now also SW62.2
- net at D30.2 (A): now also SW30.2
- net at D25.2 (A): now also SW25.2
- net at D45.2 (A): now also SW45.2
- net at D23.2 (A): now also SW23.2
- net at D37.2 (A): now also SW37.2
- net at D26.2 (A): now also SW26.2
- net at D27.2 (A): now also SW27.2
- net at D52.2 (A): now also SW52.2
- net at D16.2 (A): now also SW16.2
- net at D29.2 (A): now also SW29.2
- net at D44.2 (A): now also SW44.2
- net at D20.2 (A): now also SW20.2
- net at D55.2 (A): now also SW55.2
- net at D54.2 (A): now also SW54.2
- net at D47.2 (A): now also SW47.2
- net at D11.2 (A): now also SW11.2
- net at D10.2 (A): now also SW10.2
- net at D61.2 (A): now also SW61.2
- net at D57.2 (A): now also SW57.2
- net at D53.2 (A): now also SW53.2
- net at D56.2 (A): now also SW56.2
- net at D28.2 (A): now also SW28.2
- net at D41.2 (A): now also SW41.2
- net at D19.2 (A): now also SW19.2
- net at D63.2 (A): now also SW63.2
- net at D3.2 (A): now also SW3.2
- net VDD: now reaches C2.1, L1.2, TP2.1, U1.28 (VDD)
- net VDD: now also R4.1
- net at D7.2 (A): now also SW7.2
- net at D33.2 (A): now also SW33.2
- net at D49.2 (A): now also SW49.2
- net at D46.2 (A): now also SW46.2
- net at D40.2 (A): now also SW40.2
- net at D6.2 (A): now also SW6.2
- net at D14.2 (A): now also SW14.2
- net at D50.2 (A): now also SW50.2
- net at D35.2 (A): now also SW35.2
- net at D39.2 (A): now also SW39.2
- net at D58.2 (A): now also SW58.2
- net at D21.2 (A): now also SW21.2
- net at D24.2 (A): now also SW24.2
- net at D34.2 (A): now also SW34.2
- net at D15.2 (A): now also SW15.2
- net at D42.2 (A): now also SW42.2
- net at D43.2 (A): now also SW43.2
- net at D60.2 (A): now also SW60.2
- net at D48.2 (A): now also SW48.2
- net ofeature_enable: now reaches U1.8 (P1.15_LF)
- net ofeature_enable: now also JP1.2 (B), R4.2
- net at D8.2 (A): now also SW8.2
- net at D5.2 (A): now also SW5.2
- net at D32.2 (A): now also SW32.2
- net at D31.2 (A): now also SW31.2
- net at D12.2 (A): now also SW12.2
- net at D13.2 (A): now also SW13.2
- net at D4.2 (A): now also SW4.2
- net at D18.2 (A): now also SW18.2
- net at D36.2 (A): now also SW36.2
- net at D1.2 (A): now also SW1.2
- net at D22.2 (A): now also SW22.2
- no-connect marks 27 -> 26
